Commit message: fix: rename joints, fix mesh paths, add ros2_control tags, add controllers.yaml, update CMakeLists

File: src/scara/urdf/urdf_to_sdf_gazebo.urdf (robot description, URDF)
Before this commit: robot urdf_to_sdf_gazebo, 7 links, 6 joints
Links:
- removed link z-axis_top_plate_link_1
- added link z_axis_top_plate_link_1, mass 4.175380318770853; collision mesh filename=package://scara/meshes/z-axis_top_plate_link_1.stl scale=0.001 0.001 0.001; visual mesh filename=package://scara/meshes/z-axis_top_plate_link_1.stl scale=0.001 0.001 0.001
- link arm_cover_link_1: geometry collision mesh filename=package://scara/meshes/arm_cover_link_1.stl scale=0.001 0.001 0.001; visual mesh filename=package://scara/meshes/arm_cover_link_1.stl scale=0.001 0.001 0.001
- link arm_two_cover_link_1: geometry collision mesh filename=package://scara/meshes/arm_two_cover_link_1.stl scale=0.001 0.001 0.001; visual mesh filename=package://scara/meshes/arm_two_cover_link_1.stl scale=0.001 0.001 0.001
- link base_link: geometry collision mesh filename=package://scara/meshes/base_link.stl scale=0.001 0.001 0.001; visual mesh filename=package://scara/meshes/base_link.stl scale=0.001 0.001 0.001
- link gripper_handleftlink_1: geometry collision mesh filename=package://scara/meshes/gripper_handleftlink_1.stl scale=0.001 0.001 0.001; visual mesh filename=package://scara/meshes/gripper_handleftlink_1.stl scale=0.001 0.001 0.001
- link gripper_mechanismslider_link_1: geometry collision mesh filename=package://scara/meshes/gripper_mechanismslider_link_1.stl scale=0.001 0.001 0.001; visual mesh filename=package://scara/meshes/gripper_mechanismslider_link_1.stl scale=0.001 0.001 0.001
- link gripper_rail_6mm_bottom_link_1: geometry collision mesh filename=package://scara/meshes/gripper_rail_6mm_bottom_link_1.stl scale=0.001 0.001 0.001; visual mesh filename=package://scara/meshes/gripper_rail_6mm_bottom_link_1.stl scale=0.001 0.001 0.001
Joints:
- removed joint Revolute 10
- removed joint Revolute 7
- removed joint Revolute 8
- removed joint Slider 11
- removed joint Slider 4
- removed joint Slider 5
- added joint joint1: type revolute, parent base_link, child z_axis_top_plate_link_1, origin xyz=0.041226 -9.1e-05 0.033561 rpy=0 0 0, axis 0.0 0.0 1.0, limit lower=-2.356194 upper=2.007129 effort=100 velocity=100
- added joint joint2: type revolute, parent arm_cover_link_1, child arm_two_cover_link_1, origin xyz=0.194258 0.016995 -0.0445 rpy=0 0 0, axis 0.0 0.0 1.0, limit lower=-3.316126 upper=1.570796 effort=100 velocity=100
- added joint joint3: type prismatic, parent z_axis_top_plate_link_1, child arm_cover_link_1, origin xyz=0.03325 0.002304 0.231289 rpy=0 0 0, axis 0.0 0.0 -1.0, limit lower=-0.13 upper=0.1 effort=100 velocity=100
- added joint joint4: type revolute, parent arm_two_cover_link_1, child gripper_rail_6mm_bottom_link_1, origin xyz=0.080764 0.109723 -0.057713 rpy=0 0 0, axis -0.0 0.0 1.0, limit lower=-0.959931 upper=2.007129 effort=100 velocity=100
- added joint joint_gripper_left: type prismatic, parent gripper_rail_6mm_bottom_link_1, child gripper_handleftlink_1, origin xyz=0.050697 0.037329 -0.033935 rpy=0 0 0, axis 0.803283 0.595598 0.0, limit lower=-0.015 upper=0.0 effort=100 velocity=100
- added joint joint_gripper_right: type prismatic, parent gripper_rail_6mm_bottom_link_1, child gripper_mechanismslider_link_1, origin xyz=-0.049713 -0.037121 -0.033935 rpy=0 0 0, axis -0.803283 -0.595598 -0.0, limit lower=-0.019 upper=0.0 effort=100 velocity=100

Commit message: fix: resolve controllers.yaml path at launch time, remove $(find) from URDF

File: src/scara/urdf/urdf_to_sdf_gazebo.urdf (robot description, URDF)
Before this commit: robot urdf_to_sdf_gazebo, 7 links, 6 joints
Joints:
- joint joint4: axis -0.0 0.0 1.0 -> 0.0 0.0 1.0

Commit message: updates people updates

File: src/scara/urdf/urdf_to_sdf_gazebo.urdf (robot description, URDF)
Before this commit: robot urdf_to_sdf_gazebo, 7 links, 6 joints
Links:
- added link world
Joints:
- added joint world_fixed: type fixed, parent world, child base_link, origin xyz=0 0 0 rpy=0 0 0
